Commit message: Add default inertia tag for simulation

File: urdf/pilsbot.urdf.xacro (robot description, xacro)
@@ -7,4 +7,11 @@
   <xacro:property name="front_wheel_length" value="0.05"/>
   <xacro:property name="rear_wheel_length" value="0.08"/>
+  <xacro:macro name="default_inertia">
+    <inertial>
+      <origin xyz="0.0 0.0 0.0" rpy="0.0 1.57 1.57"/>
+      <mass value="1.0"/>
+      <inertia ixx="1.0" ixy="0.0" ixz="0.0" iyy="1.0" iyz="0.0" izz="1.0"/>
+    </inertial>
+  </xacro:macro>
   <xacro:macro name="front_wheel" params="suffix axle_offset">
     <link name="front_wheel_${suffix}">
@@ -81,9 +88,5 @@
   <xacro:macro name="axle" params="prefix length parent *origin">
     <link name="${prefix}_axle">
-      <inertial>
-        <origin xyz="0.0 0.0 0.0" rpy="0.0 1.57 1.57"/>
-        <mass value="0.0"/>
-        <inertia ixx="0.0" ixy="0.0" ixz="0.0" iyy="0.0" iyz="0.0" izz="0.0"/>
-      </inertial>
+      <xacro:default_inertia/>
       <visual name="front_axle_vis">
         <origin xyz="0.0 0.0 0.0" rpy="0.0 1.57 1.57"/>
@@ -110,9 +113,5 @@
   <xacro:macro name="frame_bar" params="prefix parent length *origin">
     <link name="${prefix}_frame_bar">
-      <inertial>
-        <origin xyz="0.0 0.0 0.0" rpy="0.0 1.57 1.57"/>
-        <mass value="0.0"/>
-        <inertia ixx="0.0" ixy="0.0" ixz="0.0" iyy="0.0" iyz="0.0" izz="0.0"/>
-      </inertial>
+      <xacro:default_inertia/>
       <visual name="front_frame_bar_vis">
         <origin xyz="0.0 0.0 0.0" rpy="0.0 1.57 1.57"/>
@@ -156,9 +155,5 @@
   </xacro:axle>
   <link name="steering_axle">
-    <inertial>
-      <origin xyz="0.0 0.0 0.0" rpy="0.0 0.0 0.0"/>
-      <mass value="0.0"/>
-      <inertia ixx="0.0" ixy="0.0" ixz="0.0" iyy="0.0" iyz="0.0" izz="0.0"/>
-    </inertial>
+    <xacro:default_inertia/>
     <visual name="steering_axle">
       <origin xyz="0.0 0.0 0.0" rpy="0.0 0.0 0.0"/>

Commit message: Change linkage of rear_axle

File: urdf/pilsbot.urdf.xacro (robot description, xacro)
@@ -151,6 +151,6 @@
     <origin xyz="0 0 0.125" rpy="0 0 0"/>
   </xacro:axle>
-  <xacro:axle prefix="rear" length="0.5" parent="front_axle">
-    <origin xyz="-0.67 0 0" rpy="0 0 0"/>
+  <xacro:axle prefix="rear" length="0.5" parent="back_frame_bar">
+    <origin xyz="0.13 0.0 -0.15" rpy="0 0 0"/>
   </xacro:axle>
   <link name="steering_axle">

Commit message: Fix wrong limits for wheels

File: urdf/pilsbot.urdf.xacro (robot description, xacro)
@@ -41,5 +41,5 @@
       <child link="front_wheel_${suffix}"/>
       <axis xyz="0 1 0"/>
-      <limit lower="-3.14159" upper="3.14159" velocity="50.0" effort="1000.0"/>
+      <limit lower="-1e+16" upper="1e+16" velocity="50.0" effort="1000.0"/>
       <origin xyz="0 ${axle_offset} 0" rpy="0 0 0"/>
     </joint>
@@ -85,5 +85,5 @@
       <child link="rear_wheel_${suffix}"/>
       <axis xyz="0 1 0"/>
-      <limit lower="-3.14159" upper="3.14159" velocity="50.0" effort="1000.0"/>
+      <limit lower="-1e+16" upper="1e+16" velocity="50.0" effort="1000.0"/>
       <origin xyz="0 ${axle_offset} 0" rpy="0 0 0"/>
     </joint>

Commit message: Fattened bot

File: urdf/pilsbot.urdf.xacro (robot description, xacro)
@@ -18,5 +18,5 @@
       <inertial>
         <origin xyz="0.0 0.0 0.0" rpy="0.0 1.57 1.57"/>
-        <mass value="1.0"/>
+        <mass value="4.0"/>
         <inertia ixx="1.0" ixy="0.0" ixz="0.0" iyy="1.0" iyz="0.0" izz="1.0"/>
       </inertial>
@@ -94,5 +94,9 @@
   <xacro:macro name="axle" params="prefix length parent *origin">
     <link name="${prefix}_axle">
-      <xacro:default_inertia/>
+      <inertial>
+        <origin xyz="0.0 0.0 0.0" rpy="0.0 1.57 1.57"/>
+        <mass value="3.0"/>
+        <inertia ixx="1.0" ixy="0.0" ixz="0.0" iyy="1.0" iyz="0.0" izz="1.0"/>
+      </inertial>
       <visual name="">
         <origin xyz="0.0 0.0 0.0" rpy="0.0 1.57 1.57"/>
@@ -122,5 +126,9 @@
   <xacro:macro name="frame_bar" params="prefix parent length *origin">
     <link name="${prefix}_frame_bar">
-      <xacro:default_inertia/>
+      <inertial>
+        <origin xyz="0.0 0.0 0.0" rpy="0.0 1.57 1.57"/>
+        <mass value="3.0"/>
+        <inertia ixx="1.0" ixy="0.0" ixz="0.0" iyy="1.0" iyz="0.0" izz="1.0"/>
+      </inertial>
       <visual name="">
         <origin xyz="0.0 0.0 0.0" rpy="0.0 1.57 1.57"/>
@@ -167,5 +175,9 @@
   </xacro:axle>
   <link name="steering_axle">
-    <xacro:default_inertia/>
+    <inertial>
+      <origin xyz="0.0 0.0 0.0" rpy="0.0 1.57 1.57"/>
+      <mass value="10.0"/>
+      <inertia ixx="1.0" ixy="0.0" ixz="0.0" iyy="1.0" iyz="0.0" izz="1.0"/>
+    </inertial>
     <visual name="steering_axle">
       <origin xyz="0.0 0.0 0.0" rpy="0.0 0.0 0.0"/>
