Commit message: Use gazebo tag for gazebo refrences Beginners fault... 🙈

File: urdf/pilsbot.gazebo.urdf.xacro (robot description, xacro)
@@ -20,12 +20,19 @@
         </geometry>
       </collision>
+    </link>
+    <joint name="${prefix}_camera_joint" type="fixed">
+      <parent link="${parent}"/>
+      <child link="${prefix}_camera_link"/>
+      <origin xyz="0.01 0.0 0.0" rpy="0.0 0.0 0.0"/>
+    </joint>
+    <gazebo reference="${prefix}_camera_link">
       <sensor type="camera" name="${prefix}_camera">
-        <always_on>0</always_on>
+        <always_on>true</always_on>
         <update_rate>30</update_rate>
         <camera name="${prefix}_camera">
           <horizontal_fov>1.16937</horizontal_fov>
           <image>
-            <width>1920</width>
-            <height>1080</height>
+            <width>848</width>
+            <height>480</height>
           </image>
           <!-- Parameters taken from the real sensor. -->
@@ -54,31 +61,36 @@
         </plugin>
       </sensor>
-    </link>
-    <joint name="${prefix}_camera_joint" type="fixed">
-      <parent link="${parent}"/>
-      <child link="${prefix}_camera_link"/>
-      <!-- <xacro:insert_block name="origin" /> -->
-    </joint>
+      <material>Gazebo/Green</material>
+    </gazebo>
     <!-- Use gazebo_ros_joint_state_publisher instead of publishWheelJointState -->
-    <plugin name="joint_states" filename="libgazebo_ros_joint_state_publisher.so">
-      <joint_name>front_wheel_right_joint</joint_name>
-      <joint_name>front_wheel_left_joint</joint_name>
-    </plugin>
-    <plugin name='diff_drive' filename='libgazebo_ros_diff_drive.so'>
-      <ros>
-        <!-- Set namespace -->
-        <namespace>/pilsbot_velocity_controller</namespace>
-      </ros>
-      <!-- Replace camelCase elements with camel_case ones -->
-      <update_rate>50</update_rate>
-      <left_joint>front_wheel_left_joint</left_joint>
-      <right_joint>front_wheel_right_joint</right_joint>
-      <wheel_separation>0.62</wheel_separation>
-      <wheel_diameter>0.125</wheel_diameter>
-      <odometry_frame>odom_raw</odometry_frame>
-      <!-- wheelTorque and wheelAcceleration now have max_ prefix -->
-      <max_wheel_torque>20</max_wheel_torque>
-      <max_acceleration>1.0</max_acceleration>
-    </plugin>
+    <gazebo>
+      <plugin name="joint_states" filename="libgazebo_ros_joint_state_publisher.so">
+        <joint_name>front_wheel_right_joint</joint_name>
+        <joint_name>front_wheel_left_joint</joint_name>
+        <joint_name>steering_axle</joint_name>
+      </plugin>
+    </gazebo>
+    <gazebo>
+      <plugin name='diff_drive' filename='libgazebo_ros_diff_drive.so'>
+        <ros>
+          <!-- Set namespace -->
+          <namespace>/pilsbot_velocity_controller</namespace>
+        </ros>
+        <!-- Replace camelCase elements with camel_case ones -->
+        <update_rate>50</update_rate>
+        <left_joint>front_wheel_left_joint</left_joint>
+        <right_joint>front_wheel_right_joint</right_joint>
+        <wheel_separation>0.62</wheel_separation>
+        <wheel_diameter>0.125</wheel_diameter>
+        <odometry_frame>odom_raw</odometry_frame>
+        <robot_base_frame>base_link</robot_base_frame>
+        <!-- wheelTorque and wheelAcceleration now have max_ prefix -->
+        <max_wheel_torque>20</max_wheel_torque>
+        <max_acceleration>1.0</max_acceleration>
+        <publish_odom>true</publish_odom>
+        <publish_odom_tf>true</publish_odom_tf>
+        <publish_wheel_tf>true</publish_wheel_tf>
+      </plugin>
+    </gazebo>
   </xacro:macro>
 </robot>

Commit message: Colourise visuals in gazebo

File: urdf/pilsbot.gazebo.urdf.xacro (robot description, xacro)
@@ -7,5 +7,5 @@
         <inertia ixx="0.01" ixy="0.0" ixz="0.0" iyy="0.01" iyz="0.0" izz="0.01"/>
       </inertial>
-      <visual name="camera_visual">
+      <visual name="">
         <geometry>
           <box size="0.001 0.01 0.02"/>

File: urdf/pilsbot.urdf.xacro (robot description, xacro)
@@ -54,4 +54,7 @@
       </actuator>
     </transmission>
+    <gazebo reference="front_wheel_${suffix}">
+      <material>Gazebo/Black</material>
+    </gazebo>
   </xacro:macro>
   <xacro:macro name="rear_wheel" params="suffix axle_offset">
@@ -85,9 +88,12 @@
       <origin xyz="0 ${axle_offset} 0" rpy="0 0 0"/>
     </joint>
+    <gazebo reference="rear_wheel_${suffix}">
+      <material>Gazebo/Black</material>
+    </gazebo>
   </xacro:macro>
   <xacro:macro name="axle" params="prefix length parent *origin">
     <link name="${prefix}_axle">
       <xacro:default_inertia/>
-      <visual name="front_axle_vis">
+      <visual name="">
         <origin xyz="0.0 0.0 0.0" rpy="0.0 1.57 1.57"/>
         <geometry>
@@ -110,9 +116,12 @@
       <child link="${prefix}_axle" />
     </joint>
+    <gazebo reference="${prefix}_axle">
+      <material>Gazebo/Red</material>
+    </gazebo>
   </xacro:macro>
   <xacro:macro name="frame_bar" params="prefix parent length *origin">
     <link name="${prefix}_frame_bar">
       <xacro:default_inertia/>
-      <visual name="front_frame_bar_vis">
+      <visual name="">
         <origin xyz="0.0 0.0 0.0" rpy="0.0 1.57 1.57"/>
         <geometry>
@@ -135,4 +144,7 @@
       <child link="${prefix}_frame_bar" />
     </joint>
+    <gazebo reference="${prefix}_frame_bar">
+      <material>Gazebo/Red</material>
+    </gazebo>
   </xacro:macro>
   <xacro:macro name="steering_axle_bar_vis" params="prefix length *origin">
@@ -192,4 +204,7 @@
     <origin xyz="0 0 0.05" rpy="0 0 0"/>
   </joint>
+  <gazebo reference="steering_axle">
+    <material>Gazebo/Red</material>
+  </gazebo>
   <xacro:frame_bar prefix="front" parent="steering_axle" length="0.49">
     <origin xyz="0.13 0.0 0.11" rpy="0.0 0.0 0.0"/>

Commit message: now using command_controller to launch acker_diff_controller

File: urdf/pilsbot.gazebo.urdf.xacro (robot description, xacro)
@@ -66,4 +66,6 @@
     <gazebo>
       <plugin name="joint_states" filename="libgazebo_ros_joint_state_publisher.so">
+        <joint_name>front_wheel_right_joint</joint_name>
+        <joint_name>front_wheel_left_joint</joint_name>
         <joint_name>rear_wheel_right_joint</joint_name>
         <joint_name>rear_wheel_left_joint</joint_name>
@@ -72,24 +74,28 @@
     </gazebo>
     <gazebo>
-      <plugin name='diff_drive' filename='libgazebo_ros_diff_drive.so'>
+	<!--
+      <plugin name='acker_drive' filename='libgazebo_ros_diff_drive.so'>
         <ros>
-          <!-- Set namespace -->
           <namespace>/pilsbot_velocity_controller</namespace>
         </ros>
-        <!-- Replace camelCase elements with camel_case ones -->
         <update_rate>50</update_rate>
         <left_joint>front_wheel_left_joint</left_joint>
         <right_joint>front_wheel_right_joint</right_joint>
+        <axle_joint>steering_axle_joint</axle_joint>
         <wheel_separation>0.62</wheel_separation>
         <wheel_diameter>0.125</wheel_diameter>
         <odometry_frame>odom_raw</odometry_frame>
         <robot_base_frame>base_link</robot_base_frame>
-        <!-- wheelTorque and wheelAcceleration now have max_ prefix -->
         <max_wheel_torque>20</max_wheel_torque>
         <max_acceleration>1.0</max_acceleration>
+        <max_steering_angle>85</max_steering_angle>
         <publish_odom>true</publish_odom>
         <publish_odom_tf>true</publish_odom_tf>
         <publish_wheel_tf>true</publish_wheel_tf>
       </plugin>
+    -->
+    <plugin name="gazebo_ros_control" filename="libgazebo_ros_control.so">
+            <robotNamespace>/pilsbot_velocity_controller</robotNamespace>
+    </plugin>
     </gazebo>
   </xacro:macro>

File: urdf/pilsbot.urdf.xacro (robot description, xacro)
@@ -213,5 +213,5 @@
     <child link="steering_axle"/>
     <axis xyz="0 0 1"/>
-    <limit lower="-3.14159" upper="3.14159" velocity="50.0" effort="1000.0"/>
+    <limit lower="-1.58" upper="1.58" velocity="50.0" effort="1000.0"/>
     <origin xyz="0 0 0.05" rpy="0 0 0"/>
   </joint>
@@ -236,4 +236,9 @@
   <xacro:rear_wheel suffix="right" axle_offset="-0.27"/>
   <xacro:include filename="$(find pilsbot_description)/urdf/pilsbot.gazebo.urdf.xacro"/>
+  <xacro:include filename="$(find pilsbot_description)/urdf/pilsbot.ros2_control.urdf.xacro"/>
+  <xacro:pilsbot_system
+    name="PilsBotSystem"
+    use_fake_hardware="true"
+  />
   <xacro:pilsbot_gazebo prefix="front" parent="front_frame_bar" />
 </robot>

Commit message: Use correct gazebo plugin for ros2 control

File: urdf/pilsbot.gazebo.urdf.xacro (robot description, xacro)
@@ -63,39 +63,9 @@
       <material>Gazebo/Green</material>
     </gazebo>
-    <!-- Use gazebo_ros_joint_state_publisher instead of publishWheelJointState -->
     <gazebo>
-      <plugin name="joint_states" filename="libgazebo_ros_joint_state_publisher.so">
-        <joint_name>front_wheel_right_joint</joint_name>
-        <joint_name>front_wheel_left_joint</joint_name>
-        <joint_name>rear_wheel_right_joint</joint_name>
-        <joint_name>rear_wheel_left_joint</joint_name>
-        <joint_name>steering_axle_joint</joint_name>
+      <plugin name="gazebo_ros_control" filename="libgazebo_ros2_control.so">
+        <!-- Change config here! TODO: make param -->
+        <parameters>$(find pilsbot_control)/config/acker_diff_controller.yaml</parameters>
       </plugin>
-    </gazebo>
-    <gazebo>
-	<!--
-      <plugin name='acker_drive' filename='libgazebo_ros_diff_drive.so'>
-        <ros>
-          <namespace>/pilsbot_velocity_controller</namespace>
-        </ros>
-        <update_rate>50</update_rate>
-        <left_joint>front_wheel_left_joint</left_joint>
-        <right_joint>front_wheel_right_joint</right_joint>
-        <axle_joint>steering_axle_joint</axle_joint>
-        <wheel_separation>0.62</wheel_separation>
-        <wheel_diameter>0.125</wheel_diameter>
-        <odometry_frame>odom_raw</odometry_frame>
-        <robot_base_frame>base_link</robot_base_frame>
-        <max_wheel_torque>20</max_wheel_torque>
-        <max_acceleration>1.0</max_acceleration>
-        <max_steering_angle>85</max_steering_angle>
-        <publish_odom>true</publish_odom>
-        <publish_odom_tf>true</publish_odom_tf>
-        <publish_wheel_tf>true</publish_wheel_tf>
-      </plugin>
-    -->
-    <plugin name="gazebo_ros_control" filename="libgazebo_ros_control.so">
-            <robotNamespace>/pilsbot_velocity_controller</robotNamespace>
-    </plugin>
     </gazebo>
   </xacro:macro>

File: urdf/pilsbot.ros2_control.urdf.xacro (robot description, xacro)
@@ -28,4 +28,12 @@
         <state_interface name="velocity"/>
       </joint>
+      <joint name="rear_wheel_left_joint">
+        <state_interface name="position"/>
+        <state_interface name="velocity"/>
+      </joint>
+      <joint name="rear_wheel_right_joint">
+        <state_interface name="position"/>
+        <state_interface name="velocity"/>
+      </joint>
       <joint name="steering_axle_joint">
         <state_interface name="position"/>

File: urdf/pilsbot.urdf.xacro (robot description, xacro)
@@ -235,5 +235,4 @@
   <xacro:rear_wheel suffix="left" axle_offset="0.27"/>
   <xacro:rear_wheel suffix="right" axle_offset="-0.27"/>
-  <xacro:include filename="$(find pilsbot_description)/urdf/pilsbot.gazebo.urdf.xacro"/>
   <xacro:include filename="$(find pilsbot_description)/urdf/pilsbot.ros2_control.urdf.xacro"/>
   <xacro:pilsbot_system
@@ -241,4 +240,5 @@
     use_fake_hardware="true"
   />
+  <xacro:include filename="$(find pilsbot_description)/urdf/pilsbot.gazebo.urdf.xacro"/>
   <xacro:pilsbot_gazebo prefix="front" parent="front_frame_bar" />
 </robot>

Commit message: Add xacro arguments for configurable properties

File: urdf/pilsbot.gazebo.urdf.xacro (robot description, xacro)
@@ -1,5 +1,5 @@
 <?xml version="1.0"?>
 <robot xmlns:xacro="http://www.ros.org/wiki/xacro">
-  <xacro:macro name="pilsbot_gazebo" params="prefix parent">
+  <xacro:macro name="pilsbot_gazebo" params="prefix parent config">
     <link name="${prefix}_camera_link">
       <inertial>
@@ -65,6 +65,5 @@
     <gazebo>
       <plugin name="gazebo_ros_control" filename="libgazebo_ros2_control.so">
-        <!-- Change config here! TODO make param -->
-        <parameters>$(find pilsbot_control)/config/acker_diff_controller.yaml</parameters>
+        <parameters>$(find pilsbot_control)/config/${config}.yaml</parameters>
       </plugin>
     </gazebo>

File: urdf/pilsbot.ros2_control.urdf.xacro (robot description, xacro)
@@ -1,5 +1,5 @@
 <?xml version="1.0"?>
 <robot xmlns:xacro="http://www.ros.org/wiki/xacro">
-  <xacro:macro name="pilsbot_system" params="name use_fake_hardware:=^|true">
+  <xacro:macro name="pilsbot_system" params="name use_fake_hardware:=^|true hoverboard_tty_device head_mcu_tty_device wheel_radius">
     <ros2_control name="${name}" type="system">
       <hardware>
@@ -12,7 +12,7 @@
           <!-- also, especially the ports & retries, they would fit -->
           <!-- much better into a yaml file -->
-          <param name="hoverboard_tty_device">/dev/ttyS0</param>
-          <param name="head_mcu_tty_device">/dev/ttyACM0</param>
-          <param name="wheel_radius">0.125</param>
+          <param name="hoverboard_tty_device">${hoverboard_tty_device}</param>
+          <param name="head_mcu_tty_device">${head_mcu_tty_device}</param>
+          <param name="wheel_radius">${wheel_radius}</param>
         </xacro:unless>
       </hardware>
@@ -45,13 +45,13 @@
       </joint>
       <sensor name="hoverboard_api">
-		<state_interface name="voltage"/>
-		<state_interface name="avg_amperage_motor.0"/>
-		<state_interface name="avg_amperage_motor.1"/>
-		<state_interface name="tx_bufferlevel"/>
+        <state_interface name="voltage"/>
+        <state_interface name="avg_amperage_motor.0"/>
+        <state_interface name="avg_amperage_motor.1"/>
+        <state_interface name="tx_bufferlevel"/>
       </sensor>
       <sensor name="head_mcu">
-		<state_interface name="steering_angle_raw"/>
-		<state_interface name="endstop_l"/>
-		<state_interface name="endstop_r"/>
+        <state_interface name="steering_angle_raw"/>
+        <state_interface name="endstop_l"/>
+        <state_interface name="endstop_r"/>
       </sensor>
     </ros2_control>

File: urdf/pilsbot.urdf.xacro (robot description, xacro)
@@ -1,4 +1,8 @@
 <?xml version="1.0"?>
 <robot xmlns:xacro="http://www.ros.org/wiki/xacro" name="pilsbot">
+  <xacro:arg name="controller_config" default="acker_diff_controller"/>
+  <xacro:arg name="use_fake_hardware" default="true"/>
+  <xacro:arg name="hoverboard_tty_device" default="/dev/ttyS0"/>
+  <xacro:arg name="head_mcu_tty_device" default="/dev/ttyACM0"/>
   <xacro:property name="frame_length" value="0.94"/>
   <xacro:property name="frame_width" value="0.49"/>
@@ -235,10 +239,12 @@
   <xacro:rear_wheel suffix="left" axle_offset="0.27"/>
   <xacro:rear_wheel suffix="right" axle_offset="-0.27"/>
-  <xacro:include filename="$(find pilsbot_description)/urdf/pilsbot.gazebo.urdf.xacro"/>
+  <xacro:include filename="$(find pilsbot_description)/urdf/pilsbot.gazebo.urdf.xacro"
+                 config="$(arg controller_config)"/>
   <xacro:include filename="$(find pilsbot_description)/urdf/pilsbot.ros2_control.urdf.xacro"/>
-  <xacro:pilsbot_system
-    name="PilsBotSystem"
-    use_fake_hardware="false"
-  />
+  <xacro:pilsbot_system name="PilsbotSystem"
+                        use_fake_hardware="$(arg use_fake_hardware)"
+                        hoverboard_tty_device="$(arg hoverboard_tty_device)"
+                        head_mcu_tty_device="$(arg head_mcu_tty_device)"
+                        wheel_radius="${wheel_radius}"/>
   <xacro:pilsbot_gazebo prefix="front" parent="front_frame_bar" />
 </robot>

Commit message: Update gazebo model for oak-d lite

File: urdf/pilsbot.gazebo.urdf.xacro (robot description, xacro)
@@ -54,7 +54,5 @@
             <namespace></namespace>
           </ros>
-          <!-- Set camera name. If empty, defaults to sensor name (i.e. "sensor_name") -->
           <camera_name>${prefix}_camera</camera_name>
-          <!-- Set TF frame name. If empty, defaults to link name (i.e. "link_name") -->
           <frame_name>${prefix}_camera_link</frame_name>
           <hack_baseline>0.07</hack_baseline>
@@ -63,6 +61,8 @@
       <material>Gazebo/Green</material>
     </gazebo>
-    <gazebo reference="oak-d_frame">
-      <sensor type="multicamera" name="oak-d-lite">
+  <gazebo reference="oak_left_camera_frame">
+      <sensor type="camera" name="left">
+        <always_on>true</always_on>
+        <update_rate>30</update_rate>
         <camera name="left">
           <horizontal_fov>1.2741</horizontal_fov>
@@ -72,14 +72,20 @@
             <format>L8</format>
           </image>
-          <clip>
-            <near>0.3</near>
-            <far>35</far>
-          </clip>
-          <noise>
-            <type>gaussian</type>
-            <mean>0.0</mean>
-            <stddev>0.007</stddev>
-          </noise>
         </camera>
+        <plugin name="plugin_name" filename="libgazebo_ros_camera.so">
+          <ros>
+            <namespace>oak_d</namespace>
+          </ros>
+          <camera_name>left</camera_name>
+          <frame_name>oak_left_camera_optical_frame</frame_name>
+          <hack_baseline>0.075</hack_baseline>
+        </plugin>
+      </sensor>
+      <material>Gazebo/Black</material>
+    </gazebo>
+    <gazebo reference="oak_right_camera_frame">
+      <sensor type="camera" name="right">
+        <always_on>true</always_on>
+        <update_rate>30</update_rate>
         <camera name="right">
           <horizontal_fov>1.2741</horizontal_fov>
@@ -89,25 +95,15 @@
             <format>L8</format>
           </image>
-          <clip>
-            <near>0.3</near>
-            <far>35</far>
-          </clip>
-          <noise>
-            <type>gaussian</type>
-            <mean>0.0</mean>
-            <stddev>0.007</stddev>
-          </noise>
         </camera>
-        <!-- Set update_rate only sensor, not on plugin -->
-        <update_rate>30</update_rate>
-        <plugin name="oak_d_lite_stereo" filename="libgazebo_ros_camera.so">
+        <plugin name="plugin_name" filename="libgazebo_ros_camera.so">
           <ros>
-            <namespace></namespace>
+            <namespace>oak_d</namespace>
           </ros>
-          <camera_name>oak_d</camera_name>
-          <frame_name>oak_left_camera_optical_frame</frame_name>
-          <hack_baseline>0.75</hack_baseline>
+          <camera_name>right</camera_name>
+          <frame_name>oak_right_camera_optical_frame</frame_name>
+          <hack_baseline>0.075</hack_baseline>
         </plugin>
       </sensor>
+      <material>Gazebo/Black</material>
     </gazebo>
     <gazebo>

File: urdf/pilsbot.urdf.xacro (robot description, xacro)
@@ -9,7 +9,7 @@
     <xacro:arg name="base_frame"    default="oak-d_frame" />
     <xacro:arg name="parent_frame"  default="front_frame_bar" />
-    <xacro:arg name="cam_pos_x"     default="0.0" />
+    <xacro:arg name="cam_pos_x"     default="0.02" />
     <xacro:arg name="cam_pos_y"     default="0.0" />
-    <xacro:arg name="cam_pos_z"     default="0.0" />
+    <xacro:arg name="cam_pos_z"     default="0.01" />
     <xacro:arg name="cam_roll"      default="0.0" />
     <xacro:arg name="cam_pitch"     default="0.0" />
